Commit message: Etapa 3 (3a): integración TurtleBot3 Burger multi-robot con el UR5e
El TurtleBot3 Burger coexiste con el UR5e en el mundo Webots (DEF TURTLEBOT en el
dock = sitio de descarga del UR5e). Verificado en vivo: ambos robots conectan, el
UR5e hace pick&place, los controladores de ambos quedan `active`, el TurtleBot se
mueve por /cmd_vel (odom 0->0.197) y el lidar /scan publica.

Integración multi-robot (gotchas no obvios resueltos):
- namespace /tb en el driver del TurtleBot: evita el choque del /robot_description
  GLOBAL que crasheaba al UR5e ("Cannot find Motor right wheel motor").
- rsp explícito (namespace tb) publica /tb/robot_description; set_robot_state_publisher:False.
- URDF del TurtleBot con árbol mínimo COMPLETO + joints de rueda reales: sin ellos
  el parser de ros2_control falla ("Joint not found") -> exit 250 y sim congelada.
- ros2control_turtlebot.yml con claves prefijadas tb/ (si no: "type param not defined").
- sin respawn en el driver: evita re-disparo de WaitForControllerConnection
  ("executed more than once" -> shutdown en cascada).
- frames tb_ (tb_base_link/tb_odom/tb_base_scan): no chocan con base_link del UR5e.

Falta Nav2 (3b): mapa libre creado (config/mapa_libre.*); pendiente el bringup de
Nav2 (namespace /tb, map->tb_odom estático) + cableado del orquestador para llevar
la caja a la estación.

Co-Authored-By: Claude Opus 4.8 <noreply@anthropic.com>

File: urdf/turtlebot_webots.urdf (robot description, URDF)
Before this commit: robot TurtleBot3 Burger Webots, 0 links, 0 joints
Links:
- added link left_wheel_link
- added link right_wheel_link
- added link tb_base_footprint
- added link tb_base_link
- added link tb_base_scan
Joints:
- added joint left wheel motor: type continuous, parent tb_base_link, child left_wheel_link, origin xyz=0 0.08 0 rpy=0 0 0, axis 0 1 0
- added joint right wheel motor: type continuous, parent tb_base_link, child right_wheel_link, origin xyz=0 -0.08 0 rpy=0 0 0, axis 0 1 0
- added joint tb_footprint_joint: type fixed, parent tb_base_link, child tb_base_footprint, origin xyz=0 0 0 rpy=0 0 0
- added joint tb_scan_joint: type fixed, parent tb_base_link, child tb_base_scan, origin xyz=0 0 0.18 rpy=0 0 0
